File: XimeTron/XT-02_Eyecillator/XT-02_Eyecillator.brd (EAGLE design)
At the start: 50.5 x 88.9 mm, 17 parts, among them IC1 4093N

Commit message: VauxFlores XimeTron 02 Eyecillator Eagle Files
Parts:
- D1: value 1N4004 -> 1N4001
Changed lines of the file:
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@@
 <attribute name="VALUE" x="41.529" y="42.164" size="1.27" layer="27" ratio="10" rot="R180"/>
 </element>
-<element name="D1" library="diode" library_urn="urn:adsk.eagle:library:210" package="DO41-10" package3d_urn="urn:adsk.eagle:package:43336/1" value="1N4004" x="39.37" y="69.85" smashed="yes" rot="R270">
+<element name="D1" library="diode" library_urn="urn:adsk.eagle:library:210" package="DO41-10" package3d_urn="urn:adsk.eagle:package:43336/1" value="1N4001" x="39.37" y="69.85" smashed="yes" rot="R270">
 <attribute name="NAME" x="41.021" y="71.882" size="1.27" layer="25" ratio="10" rot="R270"/>
 <attribute name="VALUE" x="36.576" y="71.882" size="1.27" layer="27" ratio="10" rot="R270"/>

Commit message: Add files via upload
Parts:
- D1: value 1N4001 -> 1N4004
Connections:
- net N$8 renamed GND
Routing:
- net GND: track 132.0 -> 0.00 mm
- net N$10: track 95.4 -> 81.6 mm
- net N$6: track 87.6 -> 76.8 mm
- net N$5: track 73.7 -> 84.0 mm
- net N$4: track 59.2 -> 60.5 mm
- net N$18: track 39.4 -> 38.6 mm
- added copper zone on layer 1, net GND
- added copper zone on layer 16, net GND
