File: XimeTron/XT-02_Eyecillator/XT-02_Eyecillator.sch (EAGLE design)
At the start: 17 parts, among them IC1 4093N

Commit message: VauxFlores XimeTron 02 Eyecillator Eagle Files
Parts:
- D1: value 1N4004 -> 1N4001
Changed lines of the file:
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@@
 <part name="H4" library="holes" library_urn="urn:adsk.eagle:library:237" deviceset="MOUNT-HOLE" device="3.0" package3d_urn="urn:adsk.eagle:package:14277/1" value="MOUNT-HOLE3.0"/>
 <part name="C1" library="rcl" library_urn="urn:adsk.eagle:library:334" deviceset="CPOL-US" device="E2,5-6E" package3d_urn="urn:adsk.eagle:package:23430/1" value="100uf"/>
-<part name="D1" library="diode" library_urn="urn:adsk.eagle:library:210" deviceset="1N4004" device="" package3d_urn="urn:adsk.eagle:package:43336/1"/>
+<part name="D1" library="diode" library_urn="urn:adsk.eagle:library:210" deviceset="1N4004" device="" package3d_urn="urn:adsk.eagle:package:43336/1" value="1N4001"/>
 <part name="OUTPUT" library="thonkiconn" deviceset="WQP-PJ301M-12_JACK" device=""/>
 <part name="C2" library="rcl" library_urn="urn:adsk.eagle:library:334" deviceset="C-US" device="050-025X075" package3d_urn="urn:adsk.eagle:package:23637/1" value="10uf"/>

Commit message: Add files via upload
Parts:
- D1: value 1N4001 -> 1N4004
Connections:
- net N$8 renamed GND
Changed lines of the file:
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@@
 <part name="R2" library="rcl" library_urn="urn:adsk.eagle:library:334" deviceset="R-US_" device="0207/7" package3d_urn="urn:adsk.eagle:package:23493/2" value="22k"/>
 <part name="R3" library="rcl" library_urn="urn:adsk.eagle:library:334" deviceset="R-US_" device="0207/7" package3d_urn="urn:adsk.eagle:package:23493/2" value="22k"/>
-<part name="GND1" library="supply1" library_urn="urn:adsk.eagle:library:371" deviceset="GND" device=""/>
 <part name="POWER" library="thonkiconn" deviceset="WQP-PJ301M-12_JACK" device=""/>
 <part name="H1" library="holes" library_urn="urn:adsk.eagle:library:237" deviceset="MOUNT-HOLE" device="3.0" package3d_urn="urn:adsk.eagle:package:14277/1" value="MOUNT-HOLE3.0"/>
@@
 <part name="H4" library="holes" library_urn="urn:adsk.eagle:library:237" deviceset="MOUNT-HOLE" device="3.0" package3d_urn="urn:adsk.eagle:package:14277/1" value="MOUNT-HOLE3.0"/>
 <part name="C1" library="rcl" library_urn="urn:adsk.eagle:library:334" deviceset="CPOL-US" device="E2,5-6E" package3d_urn="urn:adsk.eagle:package:23430/1" value="100uf"/>
-<part name="D1" library="diode" library_urn="urn:adsk.eagle:library:210" deviceset="1N4004" device="" package3d_urn="urn:adsk.eagle:package:43336/1" value="1N4001"/>
+<part name="D1" library="diode" library_urn="urn:adsk.eagle:library:210" deviceset="1N4004" device="" package3d_urn="urn:adsk.eagle:package:43336/1"/>
 <part name="OUTPUT" library="thonkiconn" deviceset="WQP-PJ301M-12_JACK" device=""/>
 <part name="C2" library="rcl" library_urn="urn:adsk.eagle:library:334" deviceset="C-US" device="050-025X075" package3d_urn="urn:adsk.eagle:package:23637/1" value="10uf"/>
+<part name="GND1" library="supply1" library_urn="urn:adsk.eagle:library:371" deviceset="GND" device=""/>
 </parts>
 <sheets>
@@
 <attribute name="VALUE" x="82.55" y="34.798" size="1.778" layer="96"/>
 </instance>
-<instance part="GND1" gate="1" x="73.66" y="17.78" smashed="yes">
-<attribute name="VALUE" x="71.12" y="15.24" size="1.778" layer="96"/>
-</instance>
 <instance part="POWER" gate="G$1" x="-10.16" y="78.74" smashed="yes">
 <attribute name="NAME" x="-12.7" y="82.804" size="1.778" layer="95"/>
@@
 <attribute name="NAME" x="26.416" y="33.655" size="1.778" layer="95"/>
 <attribute name="VALUE" x="26.416" y="28.829" size="1.778" layer="96"/>
+</instance>
+<instance part="GND1" gate="1" x="86.36" y="22.86" smashed="yes">
+<attribute name="VALUE" x="83.82" y="20.32" size="1.778" layer="96"/>
 </instance>
 </instances>
@@
 </segment>
 </net>
-<net name="N$8" class="0">
+<net name="GND" class="0">
 <segment>
 <pinref part="POWER" gate="G$1" pin="1"/>
@@
 <wire x1="48.26" y1="27.94" x2="73.66" y2="27.94" width="0.1524" layer="91"/>
 <junction x="48.26" y="27.94"/>
-<wire x1="157.48" y1="25.4" x2="73.66" y2="25.4" width="0.1524" layer="91"/>
+<wire x1="157.48" y1="25.4" x2="86.36" y2="25.4" width="0.1524" layer="91"/>
+<wire x1="86.36" y1="25.4" x2="73.66" y2="25.4" width="0.1524" layer="91"/>
 <wire x1="73.66" y1="25.4" x2="73.66" y2="27.94" width="0.1524" layer="91"/>
 <junction x="73.66" y="27.94"/>
-<pinref part="GND1" gate="1" pin="GND"/>
-<wire x1="73.66" y1="25.4" x2="73.66" y2="20.32" width="0.1524" layer="91"/>
-<junction x="73.66" y="25.4"/>
 <wire x1="71.12" y1="73.66" x2="134.62" y2="73.66" width="0.1524" layer="91"/>
 <pinref part="C1" gate="G$1" pin="-"/>
@@
 <wire x1="-22.86" y1="58.42" x2="-25.4" y2="58.42" width="0.1524" layer="91"/>
 <junction x="-25.4" y="58.42"/>
-</segment>
-</net>
+<pinref part="GND1" gate="1" pin="GND"/>
+<junction x="86.36" y="25.4"/>
+</segment>
+</net>
