File: Eyetron/EyeTron.sch (EAGLE design)
At the start: 40 parts, among them IC1 4093N, IC2 4093N, IC3 4093N, IC4 4077N, J1 MONOSW1GND

Commit message: Add files via upload
Connections:
- net N$34 renamed GND
Changed lines of the file:
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@@
 <part name="C6" library="rcl" library_urn="urn:adsk.eagle:library:334" deviceset="C-US" device="050-025X075" package3d_urn="urn:adsk.eagle:package:23637/1" value="10uf"/>
 <part name="C5" library="rcl" library_urn="urn:adsk.eagle:library:334" deviceset="C-US" device="050-025X075" package3d_urn="urn:adsk.eagle:package:23637/1" value="10uf"/>
+<part name="GND2" library="supply1" library_urn="urn:adsk.eagle:library:371" deviceset="GND" device=""/>
 </parts>
 <sheets>
@@
 <attribute name="NAME" x="-1.524" y="84.455" size="1.778" layer="95"/>
 <attribute name="VALUE" x="-1.524" y="79.629" size="1.778" layer="96"/>
+</instance>
+<instance part="GND2" gate="1" x="73.66" y="5.08" smashed="yes">
+<attribute name="VALUE" x="71.12" y="2.54" size="1.778" layer="96"/>
 </instance>
 </instances>
@@
 </segment>
 </net>
-<net name="N$34" class="0">
+<net name="GND" class="0">
 <segment>
 <pinref part="J1" gate="A" pin="S"/>
@@
 <wire x1="-45.72" y1="48.26" x2="-48.26" y2="48.26" width="0.1524" layer="91"/>
 <wire x1="132.08" y1="76.2" x2="132.08" y2="7.62" width="0.1524" layer="91"/>
-<wire x1="132.08" y1="7.62" x2="53.34" y2="7.62" width="0.1524" layer="91"/>
+<wire x1="132.08" y1="7.62" x2="73.66" y2="7.62" width="0.1524" layer="91"/>
 <junction x="132.08" y="76.2"/>
 <junction x="53.34" y="7.62"/>
@@
 <pinref part="C5" gate="G$1" pin="2"/>
 <junction x="-2.54" y="78.74"/>
-</segment>
-</net>
+<pinref part="GND2" gate="1" pin="GND"/>
+<wire x1="73.66" y1="7.62" x2="53.34" y2="7.62" width="0.1524" layer="91"/>
+<junction x="73.66" y="7.62"/>
+</segment>
+</net>
