File: Eurorack/Fabrica/PCB Files/VF_FabricaDeUnicorniosMuertos_PCB.sch (EAGLE design)
At the start: 23 parts, among them IC1 40106N, IC3 78l09, IC7 4066N, IC8 TL072

Commit message: Update VF_FabricaDeUnicorniosMuertos_PCB.sch
Parts:
- C14: value .01uf -> 0.01uf
Changed lines of the file:
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@@
 <?xml version="1.0" encoding="utf-8"?>
 <!DOCTYPE eagle SYSTEM "eagle.dtd">
-<eagle version="9.5.1">
+<eagle version="9.6.2">
 <drawing>
 <settings>
@@
 <part name="IC8" library="MusicThingModular" deviceset="MCP6002" device="DIL_LONG" value="TL072"/>
 <part name="C13" library="rcl" library_urn="urn:adsk.eagle:library:334" deviceset="C-US" device="050-025X075" package3d_urn="urn:adsk.eagle:package:23637/1" value=".1uf"/>
-<part name="C14" library="rcl" library_urn="urn:adsk.eagle:library:334" deviceset="C-US" device="050-025X075" package3d_urn="urn:adsk.eagle:package:23637/1" value=".01uf"/>
+<part name="C14" library="rcl" library_urn="urn:adsk.eagle:library:334" deviceset="C-US" device="050-025X075" package3d_urn="urn:adsk.eagle:package:23637/1" value="0.01uf"/>
 <part name="C15" library="rcl" library_urn="urn:adsk.eagle:library:334" deviceset="C-US" device="050-025X075" package3d_urn="urn:adsk.eagle:package:23637/1" value="0.01uf"/>
 <part name="GND6" library="supply1" library_urn="urn:adsk.eagle:library:371" deviceset="GND" device=""/>
