File: Eurorack/Fabrica/PCB Files/VF_FabricaDeUnicorniosMuertos_PCB.brd (EAGLE design)
At the start: 27.9 x 110.5 mm, 24 parts, among them IC1 40106N, IC3 78l09, IC7 4066N, IC8 TL072

Commit message: Update VF_FabricaDeUnicorniosMuertos_PCB.brd
Parts:
- C14: value .01uf -> 0.01uf
Changed lines of the file:
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@@
 <?xml version="1.0" encoding="utf-8"?>
 <!DOCTYPE eagle SYSTEM "eagle.dtd">
-<eagle version="9.5.1">
+<eagle version="9.6.2">
 <drawing>
 <settings>
@@
 <attribute name="VALUE" x="1.524" y="66.421" size="1.27" layer="27" ratio="10" rot="R90"/>
 </element>
-<element name="C14" library="rcl" library_urn="urn:adsk.eagle:library:334" package="C050-025X075" package3d_urn="urn:adsk.eagle:package:23637/1" value=".01uf" x="25.4" y="96.52" smashed="yes" rot="R90">
+<element name="C14" library="rcl" library_urn="urn:adsk.eagle:library:334" package="C050-025X075" package3d_urn="urn:adsk.eagle:package:23637/1" value="0.01uf" x="25.4" y="96.52" smashed="yes" rot="R90">
 <attribute name="SPICEPREFIX" value="C" x="62.23" y="113.03" size="1.778" layer="27" rot="R90" display="off"/>
 <attribute name="VALUE" x="23.114" y="96.901" size="1.27" layer="27" ratio="10" rot="R90"/>
